File: rfm69 breakout.brd (EAGLE design)
At the start: 30.5 x 20.3 mm, 8 parts, among them U1 RFM69HW

Commit message: Bottom screens and smaller ground plane
Parts:
- added LOGO1: OSHW-LOGOL, SparkFun-Aesthetics:OSHW-LOGO-L
Other:
- board text added: "ANT"
- board text added: "RESET"
