File: rfm69 breakout.sch (EAGLE design)
At the start: 8 parts, among them U1 RFM69HW

Commit message: Bottom screens and smaller ground plane
Parts:
- added LOGO1: OSHW-LOGOL, SparkFun-Aesthetics:OSHW-LOGOL
